File: Snowflake.sch (KiCad schematic (older format))
At the start: 12 parts, among them J1 , J2 

Commit message: updated
Parts:
- added R1, R2, R3, R4, R5: R, Resistors_SMD:R_1812, symbol R
Connections:
- net GND: now also R1.1, R2.1, R3.1, R4.1, R5.1
- net VCC: now also R1.2, R2.2, R3.2, R4.2, R5.2
Changed lines of the file:
@@
 	10150 2700 10150 2850
 Wire Wire Line
-	10150 2850 10800 2850
+	10150 2850 11150 2850
 Wire Wire Line
 	10350 2450 10700 2450
@@
 Wire Wire Line
 	10800 2100 10800 2750
+$Comp
+L R R5
+U 1 1 59EB9A05
+P 9600 1450
+F 0 "R5" V 9680 1450 50  0000 C CNN
+F 1 "R" V 9600 1450 50  0000 C CNN
+F 2 "Resistors_SMD:R_1812" V 9530 1450 50  0001 C CNN
+F 3 "" H 9600 1450 50  0001 C CNN
+	1    9600 1450
+	1    0    0    -1
+$EndComp
+$Comp
+L R R4
+U 1 1 59EB9AD3
+P 9350 1450
+F 0 "R4" V 9430 1450 50  0000 C CNN
+F 1 "R" V 9350 1450 50  0000 C CNN
+F 2 "Resistors_SMD:R_1812" V 9280 1450 50  0001 C CNN
+F 3 "" H 9350 1450 50  0001 C CNN
+	1    9350 1450
+	1    0    0    -1
+$EndComp
+$Comp
+L R R3
+U 1 1 59EB9B82
+P 9100 1450
+F 0 "R3" V 9180 1450 50  0000 C CNN
+F 1 "R" V 9100 1450 50  0000 C CNN
+F 2 "Resistors_SMD:R_1812" V 9030 1450 50  0001 C CNN
+F 3 "" H 9100 1450 50  0001 C CNN
+	1    9100 1450
+	1    0    0    -1
+$EndComp
+$Comp
+L R R2
+U 1 1 59EB9BCF
+P 8900 1450
+F 0 "R2" V 8980 1450 50  0000 C CNN
+F 1 "R" V 8900 1450 50  0000 C CNN
+F 2 "Resistors_SMD:R_1812" V 8830 1450 50  0001 C CNN
+F 3 "" H 8900 1450 50  0001 C CNN
+	1    8900 1450
+	1    0    0    -1
+$EndComp
+$Comp
+L R R1
+U 1 1 59EB9CCC
+P 8650 1450
+F 0 "R1" V 8730 1450 50  0000 C CNN
+F 1 "R" V 8650 1450 50  0000 C CNN
+F 2 "Resistors_SMD:R_1812" V 8580 1450 50  0001 C CNN
+F 3 "" H 8650 1450 50  0001 C CNN
+	1    8650 1450
+	1    0    0    -1
+$EndComp
+Wire Wire Line
+	11150 2850 11150 1400
+Wire Wire Line
+	11150 1400 9600 1400
+Wire Wire Line
+	9600 1400 9600 1300
+Connection ~ 10800 2850
+Wire Wire Line
+	9600 1300 8650 1300
+Connection ~ 9350 1300
+Connection ~ 9100 1300
+Connection ~ 8900 1300
+Wire Wire Line
+	8650 1600 9600 1600
+Connection ~ 8900 1600
+Connection ~ 9100 1600
+Connection ~ 9350 1600
+Wire Wire Line
+	9600 1600 9600 1800
+Wire Wire Line
+	9600 1800 10150 1800
+Wire Wire Line
+	10150 1800 10150 2100
+Connection ~ 10150 2100
 $EndSCHEMATC
