File: broken/Snowflake.kicad_pcb (KiCad board)
At the start: 2 copper layers, 140.2 x 174.3 mm, 190 parts, among them J1 

Commit message: updated
Parts:
- removed the 1 at (140.7, 53.0)
- removed the 1 at (37.1, 66.2)
- removed the 1 at (141.2, 77.9)
- removed the 1 at (37.6, 91.0)
- removed the 1 at (37.0, 40.8)
- removed the 1 at (140.5, 27.6)
- removed the 2 at (111.5, 53.1)
- removed the 2 at (66.3, 66.1)
- removed the 2 at (112.0, 78.0)
- removed the 2 at (66.9, 90.9)
- removed the 2 at (66.2, 40.7)
- removed the 2 at (111.3, 27.8)
- removed the 3 at (82.2, 53.1)
- removed the 3 at (95.5, 66.1)
- removed the 3 at (82.8, 77.9)
- removed the 3 at (96.1, 91.0)
- removed the 3 at (95.4, 40.8)
- removed the 3 at (82.1, 27.7)
- removed the 4 at (124.0, 159.1)
- removed the 4 at (135.3, 142.6)
- removed the 4 at (136.3, 160.7)
- removed the 4 at (125.0, 177.2)
- removed the 4 at (121.1, 142.2)
- removed the 5 at (149.2, 144.4)
- removed the 5 at (110.0, 157.3)
- removed the 5 at (111.0, 175.4)
- removed the 5 at (150.2, 162.5)
- removed the 5 at (146.4, 127.6)
- removed the 6 at (52.8, 53.1)
- removed the 6 at (124.9, 66.1)
- removed the 6 at (53.4, 77.9)
- removed the 6 at (125.5, 91.0)
- removed the 6 at (124.8, 40.8)
- removed the 6 at (52.7, 27.7)
- removed the 7 at (23.6, 53.0)
- removed the 7 at (154.2, 66.2)
- removed the 7 at (24.1, 77.9)
- removed the 7 at (154.7, 91.0)
- removed the 7 at (154.1, 40.8)
- removed the 7 at (23.4, 27.6)
- removed the 8 at (60.5, 175.2)
- removed the 8 at (56.0, 163.4)
- removed the 8 at (51.3, 151.4)
- removed the 8 at (46.9, 139.2)
- removed the 8 at (41.9, 127.1)
- removed the 8 at (37.3, 114.9)
- removed the 9 at (85.9, 189.9)
- removed the 9 at (81.4, 178.1)
- removed the 9 at (76.7, 166.1)
- removed the 9 at (72.3, 153.9)
- removed the 9 at (67.3, 141.8)
- removed the 9 at (62.7, 129.6)
- removed the ? at (104.6, 166.3)
- removed the ? at (155.6, 150.9)
- removed the ? at (74.5, 31.7)
- removed the ? at (69.1, 31.7)
- removed the ? at (71.4, 24.4)
- removed the ? at (74.0, 24.3)
- removed the ? at (157.0, 26.9)
- removed the ? at (67.2, 22.4)
- removed the ? at (77.7, 33.7)
- removed the ? at (67.2, 33.7)
- removed the ? at (77.7, 22.4)
- removed the ? at (155.3, 23.6)
- removed the ? at (153.7, 157.6)
- removed the ? at (155.3, 32.6)
- removed the ? at (81.9, 130.7)
- removed the ? at (76.9, 119.2)
- removed the ? at (103.0, 119.1)
- removed the ? at (82.4, 130.9)
- removed the ? at (95.4, 108.4)
- removed the ? at (84.4, 108.6)
- removed the ? at (97.4, 131.1)
- removed the ? at (153.7, 147.1)
- removed the ? at (75.3, 115.8)
- removed the ? at (78.7, 110.0)
- removed the ? at (86.5, 105.5)
- removed the ? at (93.2, 105.5)
- removed the ? at (101.0, 110.0)
- removed the ? at (104.3, 115.7)
- removed the ? at (104.3, 124.8)
- removed the ? at (101.0, 130.6)
- removed the ? at (93.2, 135.1)
- removed the ? at (86.5, 135.2)
- removed the ? at (107.6, 190.8)
- removed the ? at (78.7, 130.6)
- removed the ? at (75.3, 124.8)
- removed the ? at (107.6, 180.3)
- removed the ? at (105.7, 187.0)
- removed the ? at (105.6, 184.4)
- removed the ? at (101.7, 149.5)
- removed the ? at (101.8, 152.1)
- removed the ? at (103.8, 145.3)
- removed the ? at (104.6, 168.9)
- removed the ? at (103.7, 155.8)
- removed the ? at (43.5, 171.7)
- removed the ? at (43.5, 161.2)
- removed the ? at (41.6, 169.7)
- removed the ? at (41.6, 164.4)
- removed the ? at (37.0, 152.6)
- removed the ? at (37.0, 157.9)
- removed the ? at (39.0, 149.3)
- removed the ? at (39.0, 159.9)
- removed the ? at (34.3, 147.9)
- removed the ? at (106.6, 162.2)
- removed the ? at (34.3, 137.4)
- removed the ? at (32.4, 145.9)
- removed the ? at (32.4, 140.6)
- removed the ? at (27.9, 128.4)
- removed the ? at (27.9, 133.8)
- removed the ? at (29.8, 125.2)
- removed the ? at (29.8, 135.7)
- removed the ? at (24.9, 123.6)
- removed the ? at (24.9, 113.0)
- removed the ? at (22.9, 121.6)
- removed the ? at (106.6, 172.7)
- removed the ? at (22.9, 116.3)
- removed the ? at (155.5, 58.0)
- removed the ? at (155.5, 49.0)
- removed the ? at (77.9, 47.8)
- removed the ? at (67.3, 59.0)
- removed the ? at (77.9, 59.0)
- removed the ? at (67.4, 47.7)
- removed the ? at (157.1, 52.3)
- removed the ? at (74.1, 49.7)
- removed the ? at (71.5, 49.8)
- removed the ? at (152.7, 129.0)
- removed the ? at (69.3, 57.1)
- removed the ? at (74.6, 57.1)
- removed the ? at (103.1, 62.1)
- removed the ? at (108.5, 62.1)
- removed the ? at (106.3, 69.4)
- removed the ? at (103.7, 69.5)
- removed the ? at (20.7, 66.9)
- removed the ? at (110.4, 71.5)
- removed the ? at (99.9, 60.2)
- removed the ? at (110.5, 60.2)
- removed the ? at (152.6, 139.5)
- removed the ? at (99.9, 71.4)
- removed the ? at (22.3, 70.2)
- removed the ? at (22.3, 61.2)
- removed the ? at (156.0, 82.8)
- removed the ? at (156.0, 73.8)
- removed the ? at (78.4, 72.6)
- removed the ? at (67.9, 83.9)
- removed the ? at (78.4, 83.9)
- removed the ? at (67.9, 72.6)
- removed the ? at (157.6, 77.2)
- removed the ? at (154.6, 132.8)
- removed the ? at (74.7, 74.5)
- removed the ? at (72.0, 74.6)
- removed the ? at (69.8, 81.9)
- removed the ? at (75.2, 81.9)
- removed the ? at (103.7, 87.0)
- removed the ? at (109.0, 87.0)
- removed the ? at (106.8, 94.3)
- removed the ? at (104.2, 94.3)
- removed the ? at (21.2, 91.7)
- removed the ? at (110.9, 96.3)
- removed the ? at (154.7, 135.4)
- removed the ? at (100.4, 85.0)
- removed the ? at (111.0, 85.0)
- removed the ? at (100.4, 96.2)
- removed the ? at (22.8, 95.1)
- removed the ? at (22.8, 86.1)
- removed the ? at (22.1, 35.9)
- removed the ? at (22.1, 44.9)
- removed the ? at (99.8, 46.0)
- removed the ? at (110.3, 34.8)
- removed the ? at (99.8, 34.8)
- removed the ? at (155.7, 153.5)
- removed the ? at (110.2, 46.1)
- removed the ? at (20.5, 41.5)
- removed the ? at (103.5, 44.1)
- removed the ? at (106.1, 44.1)
- removed the ? at (108.3, 36.8)
- removed the ? at (103.0, 36.8)
- removed the ? at (18.3, 104.1)
- removed the ? at (18.3, 109.4)
- removed the ? at (20.3, 100.9)
- removed the ? at (20.3, 111.4)
- added 1: , WS2812B:WS2812B, F.Cu at (384.8, 37.0)
- added 2: , WS2812B:WS2812B, F.Cu at (355.5, 37.1)
- added 3: , WS2812B:WS2812B, F.Cu at (326.3, 37.0)
- added 6: , WS2812B:WS2812B, F.Cu at (296.9, 37.0)
- added 7: , WS2812B:WS2812B, F.Cu at (267.7, 37.0)
- added 8: , WS2812B:WS2812B, F.Cu at (235.5, 124.7)
- added 9: , WS2812B:WS2812B, F.Cu at (220.7, 150.1)
- added ?: , Big pad, F.Cu at (318.7, 41.0)
- added ?: , Tiny Edge, F.Cu at (399.6, 32.9)
- added ?: , Tiny Edge, F.Cu at (399.6, 41.9)
- added ?: , Big pad, F.Cu at (314.2, 132.5)
- added ?: , Big pad, F.Cu at (309.2, 121.0)
- added ?: , Big pad, F.Cu at (335.2, 121.0)
- added ?: , Big pad, F.Cu at (314.6, 132.8)
- added ?: , Big pad, F.Cu at (327.6, 110.2)
- added ?: , Big pad, F.Cu at (316.6, 110.4)
- added ?: , Big pad, F.Cu at (313.4, 41.0)
- added ?: , Big pad, F.Cu at (329.6, 132.9)
- added ?: , Tiny Edge, F.Cu at (307.5, 117.7)
- added ?: , Tiny Edge, F.Cu at (310.9, 111.9)
- added ?: , Tiny Edge, F.Cu at (318.7, 107.4)
- added ?: , Tiny Edge, F.Cu at (325.4, 107.3)
- added ?: , Tiny Edge, F.Cu at (333.2, 111.8)
- added ?: , Tiny Edge, F.Cu at (336.6, 117.6)
- added ?: , Tiny Edge, F.Cu at (336.6, 126.6)
- added ?: , Tiny Edge, F.Cu at (333.2, 132.5)
- added ?: , Tiny Edge, F.Cu at (325.5, 136.9)
- added ?: , Big pad, F.Cu at (315.6, 33.7)
- added ?: , Tiny Edge, F.Cu at (318.7, 137.0)
- added ?: , Tiny Edge, F.Cu at (310.9, 132.5)
- added ?: , Tiny Edge, F.Cu at (307.5, 126.7)
- added ?: , Tiny Edge, F.Cu at (239.0, 107.6)
- added ?: , Tiny Edge, F.Cu at (249.5, 107.6)
- added ?: , Big pad, F.Cu at (240.9, 105.7)
- added ?: , Big pad, F.Cu at (318.2, 33.7)
- added ?: , Big pad, F.Cu at (246.3, 105.7)
- added ?: , Big pad, F.Cu at (401.2, 36.3)
- added ?: , Tiny Edge, F.Cu at (311.5, 31.7)
- added ?: , Tiny Edge, F.Cu at (322.0, 43.0)
- added ?: , Tiny Edge, F.Cu at (311.4, 43.0)
- added ?: , Tiny Edge, F.Cu at (322.0, 31.8)
- moved ? 232.2 mm to (327.5, 119.7)
- moved J1 232.2 mm to (322.2, 127.0)
- moved ? 232.2 mm to (321.9, 121.7)
- moved 5 81.6 mm to (109.6, 58.8), turned to 30 degrees
- moved 4 42.5 mm to (124.3, 84.1), turned to 30 degrees
- moved ? 30.9 mm to (127.4, 101.4), turned to 240.6 degrees
- moved ? 25.3 mm to (131.5, 103.4), turned to 90 degrees
- moved ? 21.6 mm to (134.1, 103.4), turned to 90 degrees
- moved ? 16.1 mm to (137.9, 101.5), turned to 119.4 degrees
Routing:
- net /VCC: track 1744.7 -> 383.6 mm, vias 91 -> 21
- net /GND: track 1610.7 -> 349.4 mm, vias 92 -> 22
- net (no net): track 501.9 -> 108.5 mm
- net Net-(LED104-Pad4): track 397.8 -> 66.3 mm
- net Net-(LED101-Pad2): track 382.0 -> 63.7 mm
- net /DOUT: track 343.7 -> 68.8 mm
- net Net-(LED3-Pad4): track 189.8 -> 31.6 mm
- net Net-(LED2-Pad4): track 151.3 -> 25.2 mm
- net Net-(LED102-Pad2): track 148.7 -> 24.8 mm
- net Net-(LED4-Pad4): track 147.8 -> 24.6 mm
- net Net-(LED5-Pad4): track 147.7 -> 24.6 mm
- net Net-(LED101-Pad4): track 146.7 -> 24.5 mm
- net Net-(LED6-Pad4): track 94.0 -> 29.1 mm
Other:
- board size 140.2 x 174.3 mm -> 296.6 x 125.4 mm
- board text added: "+"
- board text added: "-"
- board text added: "G"
- board text added: "GND"
- board text added: "V"
- board text added: "VCC"
- board text added: "d"
