File: broken/Snowflake.sch (KiCad schematic (older format))
At the start: 17 parts, among them J1 , J2 

Commit message: updated
Parts:
- removed R1, R2, R3, R4, R5: R, Resistors_SMD:R_1812, symbol R
Changed lines of the file:
@@
 	1    0    0    -1
 $EndComp
+$Comp
+L Conn_01x01 J1
+U 1 1 59E942E8
+P 10500 3350
+F 0 "J1" H 10500 3450 50  0000 C CNN
+F 1 " " H 10500 3250 50  0000 C CNN
+F 2 "Pin_Headers:Pin_Header_Straight_1x01_Pitch2.54mm" H 10500 3350 50  0001 C CNN
+F 3 "" H 10500 3350 50  0001 C CNN
+	1    10500 3350
+	1    0    0    -1
+$EndComp
+$Comp
+L Conn_01x03 J2
+U 1 1 59E94446
+P 11000 2850
+F 0 "J2" H 11000 3050 50  0000 C CNN
+F 1 " " H 11000 2650 50  0000 C CNN
+F 2 "Pin_Headers:Pin_Header_Straight_1x03_Pitch2.54mm" H 11000 2850 50  0001 C CNN
+F 3 "" H 11000 2850 50  0001 C CNN
+	1    11000 2850
+	1    0    0    -1
+$EndComp
+Text Label 10800 2750 0    60   ~ 0
+VCC
+Text Label 10800 2850 0    60   ~ 0
+GND
+Text Label 10300 3350 0    60   ~ 0
+DOUT
+Text Label 10800 2950 0    60   ~ 0
+DIN
 Wire Wire Line
 	9900 2250 10350 2250
@@
 	10150 2700 10150 2850
 Wire Wire Line
-	10150 2850 11150 2850
+	10150 2850 10800 2850
 Wire Wire Line
 	10350 2450 10700 2450
@@
 Wire Wire Line
 	10700 2950 10800 2950
-$Comp
-L Conn_01x01 J1
-U 1 1 59E942E8
-P 10500 3350
-F 0 "J1" H 10500 3450 50  0000 C CNN
-F 1 " " H 10500 3250 50  0000 C CNN
-F 2 "Pin_Headers:Pin_Header_Straight_1x01_Pitch2.54mm" H 10500 3350 50  0001 C CNN
-F 3 "" H 10500 3350 50  0001 C CNN
-	1    10500 3350
-	1    0    0    -1
-$EndComp
 Wire Wire Line
 	10200 3350 10300 3350
 Wire Wire Line
 	10200 5000 10200 3350
-$Comp
-L Conn_01x03 J2
-U 1 1 59E94446
-P 11000 2850
-F 0 "J2" H 11000 3050 50  0000 C CNN
-F 1 " " H 11000 2650 50  0000 C CNN
-F 2 "Pin_Headers:Pin_Header_Straight_1x03_Pitch2.54mm" H 11000 2850 50  0001 C CNN
-F 3 "" H 11000 2850 50  0001 C CNN
-	1    11000 2850
-	1    0    0    -1
-$EndComp
-Text Label 10800 2750 0    60   ~ 0
-VCC
-Text Label 10800 2850 0    60   ~ 0
-GND
-Text Label 10300 3350 0    60   ~ 0
-DOUT
-Text Label 10800 2950 0    60   ~ 0
-DIN
 Wire Wire Line
 	10800 2100 10800 2750
-$Comp
-L R R5
-U 1 1 59EB9A05
-P 9600 1450
-F 0 "R5" V 9680 1450 50  0000 C CNN
-F 1 "R" V 9600 1450 50  0000 C CNN
-F 2 "Resistors_SMD:R_1812" V 9530 1450 50  0001 C CNN
-F 3 "" H 9600 1450 50  0001 C CNN
-	1    9600 1450
-	1    0    0    -1
-$EndComp
-$Comp
-L R R4
-U 1 1 59EB9AD3
-P 9350 1450
-F 0 "R4" V 9430 1450 50  0000 C CNN
-F 1 "R" V 9350 1450 50  0000 C CNN
-F 2 "Resistors_SMD:R_1812" V 9280 1450 50  0001 C CNN
-F 3 "" H 9350 1450 50  0001 C CNN
-	1    9350 1450
-	1    0    0    -1
-$EndComp
-$Comp
-L R R3
-U 1 1 59EB9B82
-P 9100 1450
-F 0 "R3" V 9180 1450 50  0000 C CNN
-F 1 "R" V 9100 1450 50  0000 C CNN
-F 2 "Resistors_SMD:R_1812" V 9030 1450 50  0001 C CNN
-F 3 "" H 9100 1450 50  0001 C CNN
-	1    9100 1450
-	1    0    0    -1
-$EndComp
-$Comp
-L R R2
-U 1 1 59EB9BCF
-P 8900 1450
-F 0 "R2" V 8980 1450 50  0000 C CNN
-F 1 "R" V 8900 1450 50  0000 C CNN
-F 2 "Resistors_SMD:R_1812" V 8830 1450 50  0001 C CNN
-F 3 "" H 8900 1450 50  0001 C CNN
-	1    8900 1450
-	1    0    0    -1
-$EndComp
-$Comp
-L R R1
-U 1 1 59EB9CCC
-P 8650 1450
-F 0 "R1" V 8730 1450 50  0000 C CNN
-F 1 "R" V 8650 1450 50  0000 C CNN
-F 2 "Resistors_SMD:R_1812" V 8580 1450 50  0001 C CNN
-F 3 "" H 8650 1450 50  0001 C CNN
-	1    8650 1450
-	1    0    0    -1
-$EndComp
-Wire Wire Line
-	11150 2850 11150 1400
-Wire Wire Line
-	11150 1400 9600 1400
-Wire Wire Line
-	9600 1400 9600 1300
-Connection ~ 10800 2850
-Wire Wire Line
-	9600 1300 8650 1300
-Connection ~ 9350 1300
-Connection ~ 9100 1300
-Connection ~ 8900 1300
-Wire Wire Line
-	8650 1600 9600 1600
-Connection ~ 8900 1600
-Connection ~ 9100 1600
-Connection ~ 9350 1600
-Wire Wire Line
-	9600 1600 9600 1800
-Wire Wire Line
-	9600 1800 10150 1800
-Wire Wire Line
-	10150 1800 10150 2100
-Connection ~ 10150 2100
 $EndSCHEMATC
