File: broken/upper/Snowflake.kicad_pcb (KiCad board)
At the start: 2 copper layers, 228.8 x 162.2 mm, 77 parts, among them J1 

Commit message: updated
Parts:
- removed 1 (x2), 2 (x2), 3 (x2), 6 (x2), 7 (x2), 8, 9: , WS2812B:WS2812B
- removed the ? at (82.6, 54.3)
- removed the ? at (163.5, 46.2)
- removed the ? at (163.5, 55.1)
- removed the ? at (231.6, 50.0)
- removed the ? at (226.0, 52.0)
- removed the ? at (218.3, 62.8)
- removed the ? at (213.2, 51.3)
- removed the ? at (239.3, 51.3)
- removed the ? at (218.7, 63.1)
- removed the ? at (231.7, 40.5)
- removed the ? at (220.7, 40.7)
- removed the ? at (77.3, 54.3)
- removed the ? at (233.7, 63.2)
- removed the ? at (211.6, 48.0)
- removed the ? at (215.0, 42.2)
- removed the ? at (222.8, 37.7)
- removed the ? at (229.5, 37.6)
- removed the ? at (237.3, 42.1)
- removed the ? at (240.7, 47.9)
- removed the ? at (240.6, 56.9)
- removed the ? at (237.3, 62.8)
- removed the ? at (229.5, 67.2)
- removed the ? at (79.5, 47.0)
- removed the ? at (222.8, 67.3)
- removed the ? at (215.0, 62.8)
- removed the ? at (211.6, 57.0)
- removed the ? at (151.3, 145.0)
- removed the ? at (154.7, 150.7)
- removed the ? at (162.5, 155.3)
- removed the ? at (169.2, 155.2)
- removed the ? at (177.0, 150.7)
- removed the ? at (180.3, 144.9)
- removed the ? at (180.3, 135.9)
- removed the ? at (82.1, 46.9)
- removed the ? at (176.9, 130.1)
- removed the ? at (169.1, 125.6)
- removed the ? at (162.4, 125.7)
- removed the ? at (154.6, 130.1)
- removed the ? at (151.3, 136.0)
- removed the ? at (63.1, 146.0)
- removed the ? at (73.6, 146.0)
- removed the ? at (173.3, 151.2)
- removed the ? at (165.1, 49.5)
- removed the ? at (160.3, 128.7)
- removed the ? at (171.4, 128.5)
- removed the ? at (158.4, 151.1)
- removed the ? at (178.9, 139.2)
- removed the ? at (152.9, 139.3)
- removed the ? at (157.9, 150.8)
- removed the ? at (65.1, 144.1)
- removed the ? at (70.4, 144.1)
- removed the ? at (75.4, 44.9)
- removed the ? at (165.7, 140.0)
- removed the ? at (171.2, 138.0)
- removed the ? at (85.8, 56.2)
- removed the ? at (75.3, 56.2)
- removed the ? at (85.8, 45.0)
- removed J1 (x2): , Pin_Headers:Pin_Header_Straight_1x01_Pitch2.54mm
- moved 4 72.3 mm to (124.3, 84.1)
- moved 5 72.3 mm to (109.6, 58.8)
- moved ? 72.3 mm to (137.9, 101.5)
- moved ? 72.3 mm to (127.4, 101.4)
- moved ? 72.3 mm to (134.1, 103.4)
- moved ? 72.3 mm to (131.5, 103.4)
Routing:
- net /VCC: track 654.1 -> 57.4 mm, vias 36 -> 3
- net /GND: track 596.8 -> 50.4 mm, vias 38 -> 3
- net /DOUT: track 241.5 -> 0.00 mm
- net /DIN: track 160.9 -> 0.00 mm
- net Net-(LED101-Pad2): track 111.0 -> 0.00 mm
- net (no net): track 84.8 -> 0.00 mm, vias 4 -> 0
- net Net-(LED6-Pad4): track 58.2 -> 0.00 mm
- net Net-(LED4-Pad4): track 49.3 -> 0.00 mm
- net Net-(LED5-Pad4): track 49.2 -> 0.00 mm
- net Net-(LED101-Pad4): track 48.9 -> 0.00 mm
- net Net-(LED104-Pad4): track 81.6 -> 51.0 mm
- net Net-(LED102-Pad2): track 24.8 -> 0.00 mm
- net Net-(LED3-Pad4): track 43.6 -> 19.7 mm
Other:
- board size 228.8 x 162.2 mm -> 34.6 x 49.5 mm
- board text added: "G"
- board text added: "V"
- board text removed: "1"
- board text removed: "2"
- board text removed: "3"
- board text removed: "4"
- board text removed: "5"
- board text removed: "6"
- board text removed: "V0.9 Snowflake"
- board text removed: "eag"
