File: Merged/Snowflake.kicad_pcb (KiCad board)
At the start: 2 copper layers, 168.4 x 106 mm, 45 parts, among them J1 

Commit message: changes, added esp controller
Parts:
- removed the ? at (215.2, 103.1)
- removed the ? at (215.8, 112.0)
- removed the ? at (138.3, 113.0)
- removed the ? at (127.0, 113.0)
- removed the ? at (127.8, 101.7)
- removed the ? at (138.3, 101.2)
- moved ? 0.53 mm to (127.3, 112.7)
- moved ? 0.52 mm to (233.4, 121.9)
- moved ? 0.51 mm to (215.5, 111.6)
- moved ? 0.50 mm to (137.9, 101.5)
- moved ? 0.50 mm to (241.1, 96.8)
- moved ? 0.50 mm to (218.8, 96.8)
- moved ? 0.49 mm to (127.4, 101.4)
- moved ? 0.49 mm to (215.5, 102.6)
- moved ? 0.49 mm to (137.9, 112.7)
- moved ? 0.48 mm to (244.5, 111.6)
- moved ? 0.48 mm to (226.6, 92.3)
- moved ? 0.48 mm to (241.2, 117.4)
- moved ? 0.47 mm to (233.3, 92.3)
- moved ? 0.47 mm to (226.7, 121.9)
- moved ? 0.47 mm to (244.5, 102.5)
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Routing:
- net (no net): track 44.8 -> 3.06 mm
- net /DOUT: track 148.1 -> 187.6 mm
- net /DIN: track 82.7 -> 80.4 mm
- net Net-(LED101-Pad2): track 61.5 -> 63.7 mm
- net /VCC: track 384.7 -> 383.6 mm, vias 22 -> 21
- net Net-(LED3-Pad4): track 32.3 -> 31.6 mm
- net Net-(LED104-Pad4): track 66.8 -> 66.3 mm
Other:
- board text removed: "+"
- board text removed: "-"
- board text removed: "G"
- board text removed: "GND"
- board text removed: "V"
- board text removed: "VCC"
- board text removed: "d"
